File: Hardware/Proiect.brd (EAGLE design)
At the start: 170.2 x 111.2 mm, 103 parts

Commit message: Add files via upload
Parts:
- moved TP16 1.41 mm to (158.7, 39.5)
- moved ESP32 1.00 mm to (13.0, 39.4)
Routing:
- net GND: track 1114.2 -> 798.9 mm, vias 43 -> 9
- net 3V3: track 501.9 -> 443.2 mm, vias 23 -> 8
- net VBUS: track 158.0 -> 114.4 mm, vias 9 -> 0
- net INT_RTC: track 115.6 -> 76.8 mm, vias 4 -> 2
- net EPD_BUSY: track 139.0 -> 102.2 mm, vias 9 -> 2
- net 32KHZ: track 109.1 -> 74.2 mm, vias 4 -> 2
- net SDA: track 258.9 -> 227.7 mm, vias 9 -> 5
- net MOSI: track 238.2 -> 207.0 mm, vias 13 -> 8
- net SCK: track 226.1 -> 195.0 mm, vias 9 -> 6
- net SCL: track 249.8 -> 222.8 mm, vias 8 -> 4
- net EPD_RST: track 111.1 -> 85.9 mm, vias 9 -> 2
- net MISO: track 155.7 -> 132.6 mm, vias 6 -> 7
- net RESET: track 135.1 -> 112.6 mm, vias 4 -> 3
- net SRC: track 57.0 -> 34.7 mm, vias 2 -> 0
- net GDR: track 99.6 -> 112.0 mm, vias 6 -> 0
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- added copper zone on layer 1, net GND
- added copper zone on layer 16, net GND
Other:
- outline, holes or cut-outs redrawn
